File: PCB/mainboard/mainboard.kicad_sch (KiCad schematic)
At the start: 0 parts

Commit message: STM32 Mainboard requirements for Programing and Power
Parts:
- added C10, C11, C12, C13, C14, C15, C16, C17, C18, C19, C20, C31, C32, C7, C9: 100n, Capacitor_SMD:C_0201_0603Metric_Pad0.64x0.40mm_HandSolder, symbol Device:C
- added C21, C22, C23, C24, C33, C34, C8: 1u, Capacitor_SMD:C_0201_0603Metric_Pad0.64x0.40mm_HandSolder, symbol Device:C
- added C25, C26: 18p, Capacitor_SMD:C_0201_0603Metric_Pad0.64x0.40mm_HandSolder, symbol Device:C
- added C27, C28: 15p, Capacitor_SMD:C_0201_0603Metric_Pad0.64x0.40mm_HandSolder, symbol Device:C
- added C29, C30: 2.2u, Capacitor_SMD:C_0201_0603Metric_Pad0.64x0.40mm_HandSolder, symbol Device:C
- added D3, D4, D5, D6: LED, lib:LEDC1608X70N, symbol Device:LED
- added FL1: BLM31KN601SH1L, lib:BLM31KN102BH1L, symbol BLM31KN601SH1L:BLM31KN601SH1L
- added IC1: STM32H743ZIT6, lib:QFP50P2200X2200X160-144N, symbol STM32H743ZIT6:STM32H743ZIT6
- added J1: Conn_01x02_right, Connector_JST:JST_XH_B2B-XH-AM_1x02_P2.50mm_Vertical, symbol Connector_Generic:Conn_01x02
- added J2: Conn_01x02_left, Connector_JST:JST_XH_B2B-XH-AM_1x02_P2.50mm_Vertical, symbol Connector_Generic:Conn_01x02
- added J3: Conn_01x08_Pin_left, Connector_FFC-FPC:Amphenol_F32Q-1A7x1-11008_1x08-1MP_P0.5mm_Horizontal, symbol Connector:Conn_01x08_Pin
- added J4: Conn_01x06_Pin_LED_Strip_left, Connector_FFC-FPC:Amphenol_F32Q-1A7x1-11006_1x06-1MP_P0.5mm_Horizontal, symbol Connector:Conn_01x06_Pin
- added J5: Conn_01x06_Pin_LED_Strip_right, Connector_FFC-FPC:Amphenol_F32Q-1A7x1-11006_1x06-1MP_P0.5mm_Horizontal, symbol Connector:Conn_01x06_Pin
- added J6: Conn_01x08_Pin_TOF, Connector_FFC-FPC:Amphenol_F32Q-1A7x1-11008_1x08-1MP_P0.5mm_Horizontal, symbol Connector:Conn_01x08_Pin
- added J7: Conn_02x03_Counter_Clockwise, symbol Connector_Generic:Conn_02x03_Counter_Clockwise
- added J8: Conn_01x08_Pin_right, Connector_FFC-FPC:Amphenol_F32Q-1A7x1-11008_1x08-1MP_P0.5mm_Horizontal, symbol Connector:Conn_01x08_Pin
- added J9: Conn_01x02, symbol Connector_Generic:Conn_01x02
- added R10: 270R, Resistor_SMD:R_0201_0603Metric_Pad0.64x0.40mm_HandSolder, symbol Device:R
- added R11, R12, R13, R14, R15, R16, R17, R18, R19, R20, R21, R22, R23, R24, R25, R26, R27, R28, R29, R30: 47R, Resistor_SMD:R_0201_0603Metric_Pad0.64x0.40mm_HandSolder, symbol Device:R
- added R31, R32: 10R, Resistor_SMD:R_0201_0603Metric_Pad0.64x0.40mm_HandSolder, symbol Device:R
- added R5, R6: 10k, Resistor_SMD:R_0201_0603Metric_Pad0.64x0.40mm_HandSolder, symbol Device:R
- added R7, R8, R9: 100R, Resistor_SMD:R_0201_0603Metric_Pad0.64x0.40mm_HandSolder, symbol Device:R
- added S1: 434121025816, lib:434121025816, symbol 434121025816:434121025816
- added Y1: ECS-250-8-36CKM-TR3, lib:ECS250836CKMTR3, symbol ECS-250-8-36CKM-TR3:ECS-250-8-36CKM-TR3
- added Y2: CM7V-T1A-32.768KHZ-7PF-20PPM-TA-QC, lib:CM7V32768TBQA020, symbol CM7V-T1A-32_768KHZ-7PF-20PPM-T:CM7V-T1A-32.768KHZ-7PF-20PPM-TA-QC
Connections:
- new net: D5.1 (K), R9.1
- new net: IC1.138 (BOOT0), J9.1 (Pin_1), R5.2
- new net: J6.6 (Pin_6), R30.1
- new net: J3.3 (Pin_3), R18.1
- new net: J8.7 (Pin_7), R16.1
- new net: J8.5 (Pin_5), R14.1
- new net: J6.3 (Pin_3), R27.1
- new net: J6.4 (Pin_4), R28.1
- new net: J6.5 (Pin_5), R29.1
- new net: C32.1, C33.1, C7.1, C8.1, FL1.2, IC1.32 (VREF+), IC1.33 (VDDA)
- new net: J5.3 (Pin_3), R25.1
- new net: J5.4 (Pin_4), R26.1
- new net: J8.3 (Pin_3), R12.1
- new net: D6.1 (K), R10.1
- new net: J8.2 (Pin_2), R11.1
- new net: J8.4 (Pin_4), R13.1
- new net: J8.6 (Pin_6), R15.1
- new net: J8.8 (Pin_8), R31.1
- new net: J4.4 (Pin_4), R24.1
- new net: J3.6 (Pin_6), R21.1
- new net: D3.1 (K), R7.1
- new net: J3.2 (Pin_2), R17.1
- new net: J4.3 (Pin_3), R23.1
- new net: D4.1 (K), R8.1
- new net: J3.4 (Pin_4), R19.1
- new net: J3.5 (Pin_5), R20.1
- new net: J3.8 (Pin_8), R32.1
- new net: J3.7 (Pin_7), R22.1
- new net 3.3V: C10.1, C11.1, C12.1, C13.1, C14.1, C15.1, C16.1, C17.1, C18.1, C19.1, C20.1, C21.1, C22.1, C23.1, C24.1, C31.1, C34.1, D3.2 (A), D4.2 (A), D5.2 (A), FL1.1, IC1.108 (VDD_8), IC1.121 (VDD_9), IC1.131 (VDD_10), IC1.143 (PDR_ON), IC1.144 (VDD_11), IC1.17 (VDD_1), IC1.30 (VDD_2), IC1.39 (VDD_3), IC1.52 (VDD_4), IC1.6 (VBAT), IC1.62 (VDD_5), IC1.72 (VDD_6), IC1.84 (VDD_7), IC1.95 (VDD33USB), J6.1 (Pin_1), J6.2 (Pin_2), J7.1 (Pin_1), J9.2 (Pin_2), R6.1
- new net 5V: D6.2 (A), J4.1 (Pin_1), J4.6 (Pin_6), J5.1 (Pin_1), J5.6 (Pin_6)
- new net DIN Board 1: R23.2, R24.2
- new net DIN Board 2: R25.2, R26.2
- new net GND: C10.2, C11.2, C12.2, C13.2, C14.2, C15.2, C16.2, C17.2, C18.2, C19.2, C20.2, C21.2, C22.2, C23.2, C24.2, C25.1, C26.2, C27.2, C28.2, C29.2, C30.2, C31.2, C32.2, C33.2, C34.2, C7.2, C8.2, C9.2, IC1.107 (VSS_7), IC1.120 (VSS_8), IC1.130 (VSS_9), IC1.16 (VSS_1), IC1.31 (VSSA), IC1.38 (VSS_2), IC1.51 (VSS_3), IC1.61 (VSS_4), IC1.83 (VSS_5), IC1.94 (VSS_6), J1.1 (Pin_1), J2.1 (Pin_1), J3.1 (Pin_1), J4.2 (Pin_2), J4.5 (Pin_5), J5.2 (Pin_2), J5.5 (Pin_5), J6.7 (Pin_7), J6.8 (Pin_8), J7.3 (Pin_3), J8.1 (Pin_1), R10.2, R5.1, R9.2, S1.1, Y1.2 (GND_1), Y1.4 (GND_2)
- new net GPIO 1: R27.2
- new net NRST: C9.1, IC1.25 (NRST), J7.5 (Pin_5), R6.2, S1.2
- new net PC14-OSC32_IN: C28.1, IC1.8 (PC14-OSC32_IN), Y2.1
- new net PC15-OSC32_OUT: C27.1, IC1.9 (PC15-OSC32_OUT), Y2.2
- new net PE2: IC1.1 (PE2), R8.2
- new net PF10: IC1.22 (PF10), R7.2
- new net PH0-OSC_IN: C25.2, IC1.23 (PH0-OSC_IN), Y1.1 (IN/OUT)
- new net PH1-OSC_OUT: C26.1, IC1.24 (PH1-OSC_OUT), Y1.3 (OUT/IN)
- new net SCL: R29.2
- new net SDA: R28.2
- new net SWCLK: IC1.109 (PA14), J7.4 (Pin_4)
- new net SWDIO: IC1.105 (PA13), J7.2 (Pin_2)
- new net SWo: IC1.133 (PB3), J7.6 (Pin_6)
- new net VCAP_1: C29.1, IC1.71 (VCAP_1)
- new net VCAP_2: C30.1, IC1.106 (VCAP_2)
- new net VCC: J1.2 (Pin_2), J2.2 (Pin_2)
- new net XSHUT: R30.2
- new net left_A0: R19.2
- new net left_A1: R18.2
- new net left_A2: R17.2
- new net left_ADC INPUT: R32.2
- new net left_SCL: R21.2
- new net left_SDA: R20.2
- new net left_¬EN: R22.2
- new net right_A0: R13.2
- new net right_A1: R12.2
- new net right_A2: R11.2
- new net right_ADC INPUT: R31.2
- new net right_SCL: R15.2
- new net right_SDA: R14.2
- new net right_¬EN: R16.2
Other:
- added sheet 3.3V 3 A Buck Converter (3.3V.kicad_sch)
- added sheet 5V 3A Buck Converter (5V.kicad_sch)
- note added: "Buck Converters"
- note added: "Core Voltage VCAP Decoupling"
- note added: "Debug LED's"
- note added: "Decoupling Capacitors"
- note added: "High-Speed External (HSE) Crystal Oszilator"
- note added: "LED Strip left"
- note added: "LED Strip right"
- note added: "Left Strip"
- note added: "Low-Speed External (LSE) Crystal Oszilator"
- note added: "Right Strip"
- note added: "ST-Link"
- note added: "Time Of Flight"
- company: (none) -> RRG
- title: (none) -> Mainboard Hexapod
