File: PCB/mainboard/MCU_Configuration.kicad_sch (KiCad schematic)
At the start: 14 parts, among them Y1 ECS-250-8-36CKM-TR3, Y2 CM7V-T1A-32.768KHZ-7PF-20PPM-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

Commit message: Made the Mainboard BCP Part Layout
Parts:
- removed S2, S3: 434121025816, lib:434121025816, symbol 434121025816:434121025816
- removed Y1: ECS-250-8-36CKM-TR3, lib:ECS250836CKMTR3, symbol ECS-250-8-36CKM-TR3:ECS-250-8-36CKM-TR3
- removed Y2: CM7V-T1A-32.768KHZ-7PF-20PPM-TA-QC, lib:CM7V32768TBQA020, symbol CM7V-T1A-32_768KHZ-7PF-20PPM-T:CM7V-T1A-32.768KHZ-7PF-20PPM-TA-QC
- added C9: 100n, Capacitor_SMD:C_0402_1005Metric_Pad0.74x0.62mm_HandSolder, symbol Device:C
- added R6: 10k, Resistor_SMD:R_0201_0603Metric_Pad0.64x0.40mm_HandSolder, symbol Device:R
- added S1, S4, S5: 434121025816, lib:434121025816, symbol 434121025816:434121025816
- added Y1: CM7V-T1A-32.768KHZ-7PF-20PPM-TA-QC, lib:CM7V32768TBQA020, symbol CM7V-T1A-32_768KHZ-7PF-20PPM-T:CM7V-T1A-32.768KHZ-7PF-20PPM-TA-QC
- added Y3: ECS-250-8-36CKM-TR3, lib:ECS250836CKMTR3, symbol ECS-250-8-36CKM-TR3:ECS-250-8-36CKM-TR3
Connections:
- net +3V3: now also S1.1 (COM), S5.1 (COM)
- net Boot0: now also S5.2 (NO)
- net GND: now also C9.1, R6.1, S4.2 (NO), Y3.2 (GND_1), Y3.4 (GND_2)
- net NRST: now also S4.1 (COM)
- net PC14-OSC32_IN: now also Y1.1
- net PC15-OSC32_OUT: now also Y1.2
- net PH0-OSC_IN: now also Y3.1 (IN/OUT)
- net PH1-OSC_OUT: now also Y3.3 (OUT/IN)
- new net User Button: C9.2, R6.2, S1.2 (NO)
Other:
- note added: "User Button"

Commit message: random upload
Parts:
- removed C44: 100n, Capacitor_SMD:C_0402_1005Metric_Pad0.74x0.62mm_HandSolder, symbol Device:C
- removed S5: 434121025816, lib:434121025816, symbol 434121025816:434121025816
- C25, C26: value 10pF -> 6pF
Other:
- note added: "BOOT0"
- note removed: "BOOT0 Button"
- moved on the sheet: R5
