File: PCB/mainboard/mainboard.kicad_pcb (KiCad board)
At the start: 4 copper layers, 100 x 68 mm, 131 parts, among them IC1 74HCT125T14-13, IC2 SP4065-08ATG, IC4 STM32H743ZIT6, J1 Right Strip Power, J10 Uart Connector to pi5, J11 Conn_02x05_Counter_Clockwise, J2 Left Strip Power, J3 Left Strip, J4 LED Strip left, J5 LED Strip right, J6 Time Of Flight, J7 TST-105-01-L-D, J8 Right Strip, U1 TPS5430DDA, U2 TPS5430DDA, Y1 CM7V-T1A-32.768KHZ-7PF-20PPM-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, Y3 ECS-250-8-36CKM-TR3

Commit message: random upload
Parts:
- removed C44: 100n, Capacitor_SMD:C_0402_1005Metric_Pad0.74x0.62mm_HandSolder
- removed D2, D9: B340A-13-F, lib:DIOM5226X240N
- removed L1, L3: MGAH06033R3M-10, lib:IND_MGAH06033R3M-10
- removed R39, R40: 47R, Resistor_SMD:R_0201_0603Metric_Pad0.64x0.40mm_HandSolder
- removed S5: 434121025816, lib:434121025816
- removed U1, U2: TPS5430DDA, Package_SO:TI_SO-PowerPAD-8_ThermalVias
- added C47: 10n, Capacitor_SMD:C_0402_1005Metric_Pad0.74x0.62mm_HandSolder, F.Cu at (186.2, 109.7)
- added C48: 100n, Capacitor_SMD:C_0402_1005Metric_Pad0.74x0.62mm_HandSolder, F.Cu at (187.0, 105.0)
- added C49: 10u, Capacitor_SMD:C_0402_1005Metric_Pad0.74x0.62mm_HandSolder, F.Cu at (188.0, 105.0)
- added C6: 22p, Capacitor_SMD:C_0402_1005Metric_Pad0.74x0.62mm_HandSolder, F.Cu at (183.8, 108.7)
- added R29: 27.4k, Resistor_SMD:R_0402_1005Metric_Pad0.72x0.64mm_HandSolder, F.Cu at (186.2, 108.7)
- added R33: 10k, Resistor_SMD:R_0402_1005Metric_Pad0.72x0.64mm_HandSolder, F.Cu at (183.8, 109.7)
- added R34: 135k, Resistor_SMD:R_0402_1005Metric_Pad0.72x0.64mm_HandSolder, F.Cu at (183.8, 107.7)
- added R44: 30k, Resistor_SMD:R_0402_1005Metric_Pad0.72x0.64mm_HandSolder, F.Cu at (186.2, 107.7)
- added VR1: TPSM863252RDXR, lib:VREG_TPSM863252RDXR, F.Cu at (183.9, 104.3)
- added VR2: TPSM863252RDXR, lib:VREG_TPSM863252RDXR, F.Cu at (122.0, 103.8)
- C1: footprint Capacitor_SMD:C_1206_3216Metric_Pad1.33x1.80mm_HandSolder -> Capacitor_SMD:C_0402_1005Metric_Pad0.74x0.62mm_HandSolder
- C2: value 10n -> 100n; footprint Capacitor_SMD:C_1206_3216Metric_Pad1.33x1.80mm_HandSolder -> Capacitor_SMD:C_0402_1005Metric_Pad0.74x0.62mm_HandSolder
- C25, C26: value 10pF -> 6pF
- C3: value EEE-FP0J331AV 220u -> 10n; footprint lib:EEEFP0J331AV -> Capacitor_SMD:C_0402_1005Metric_Pad0.74x0.62mm_HandSolder
- C4: value 10u -> 22p; footprint Capacitor_SMD:C_1206_3216Metric_Pad1.33x1.80mm_HandSolder -> Capacitor_SMD:C_0402_1005Metric_Pad0.74x0.62mm_HandSolder
- C46: value EEE-FP0J331AV 220u -> 33u; footprint lib:EEEFP0J331AV -> lib:C4532_Commercial
- C5: value 10n -> 33u; footprint Capacitor_SMD:C_1206_3216Metric_Pad1.33x1.80mm_HandSolder -> lib:C4532_Commercial
- R1: value 51k -> 27.4k
- R3: value 31.6k -> 220k
- R37, R38: value 330R -> 47R
- R4: value 10k -> 30k
- moved TP3 71.4 mm to (115.3, 108.5), turned to 180 degrees
- moved TP4 68.8 mm to (118.5, 108.6), turned to 180 degrees
- moved C4 66.4 mm to (121.9, 108.0), turned to 0 degrees
- moved D5 66.4 mm to (120.7, 99.8)
- moved C46 65.7 mm to (178.9, 103.4), turned to -90 degrees
- moved R9 64.2 mm to (122.1, 99.0), turned to -90 degrees
- moved R10 64.0 mm to (184.1, 99.5), turned to -90 degrees
- moved C5 63.4 mm to (116.9, 102.8), turned to -90 degrees
- moved D6 62.3 mm to (182.7, 100.3)
- moved TP2 59.0 mm to (180.5, 108.9), turned to 180 degrees
- moved R4 56.4 mm to (124.2, 107.0)
- moved R3 56.1 mm to (121.9, 107.0)
- moved TP1 55.2 mm to (177.3, 108.9), turned to 180 degrees
- moved C3 54.7 mm to (124.2, 109.0), turned to 0 degrees
- moved C41 15.0 mm to (183.9, 112.3)
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Connections:
- AC2 pad 2: unconnected-(AC2-SDX-Pad2) -> GND
- AC2 pad 3: unconnected-(AC2-SCX-Pad3) -> GND
- C2 pad 1: Net-(U1-BOOT) -> VCC
- C2 pad 2: PH 5 -> GND
- C3 pad 1: +3V3 -> Net-(VR2-EN)
- C4 pad 1: VCC -> +3V3
- C4 pad 2: GND -> Net-(VR2-FB)
- C5 pad 1: Net-(U2-BOOT) -> +3V3
- C5 pad 2: PH 3.3 -> GND
- J11 pad 8: Net-(J11-Pin_8) -> SCL
- J11 pad 9: Net-(J11-Pin_9) -> SDA
- R1 pad 1: +5V -> VCC
- R1 pad 2: Net-(U1-VSENSE) -> Net-(VR2-EN)
- R2 pad 1: Net-(U1-VSENSE) -> Net-(VR2-EN)
- R3 pad 2: Net-(U2-VSENSE) -> Net-(VR2-FB)
- R4 pad 1: Net-(U2-VSENSE) -> Net-(VR2-FB)
Routing:
- net VCC: track 107.5 -> 170.4 mm, vias 18 -> 12
- net Net-(VR1-EN): track 0.00 -> 11.4 mm
- net Net-(VR2-EN): track 0.00 -> 10.6 mm
- net Net-(J11-Pin_8): track 6.90 -> 0.00 mm
- net +3V3: track 69.6 -> 76.1 mm, vias 57 -> 38
- net GND: track 1.46 -> 7.77 mm, vias 170 -> 88
- net SDA: track 206.2 -> 199.9 mm
- net left_A2: track 44.9 -> 39.3 mm
- net left_A1: track 44.3 -> 39.0 mm
- net right_A0: track 44.9 -> 50.2 mm
- net right_¬EN: track 56.4 -> 61.7 mm
- net right_A1: track 45.0 -> 50.2 mm
- net Boot0: track 7.20 -> 2.08 mm
- net right_A2: track 44.8 -> 49.9 mm
- net XSHUT: track 52.0 -> 56.9 mm
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- removed copper zone on F.Cu, net PH 3.3
- removed copper zone on F.Cu, net PH 5
Other:
- outline, holes or cut-outs redrawn
- board text added: "NRST"
- board text added: "User Buttom"

Commit message: random
Parts:
- added J9: LED_CAM, Connector_PinHeader_2.54mm:PinHeader_1x02_P2.54mm_Vertical, F.Cu at (160.8, 83.0)
- added R39: 100R, Resistor_SMD:R_0201_0603Metric_Pad0.64x0.40mm_HandSolder, F.Cu at (160.3, 87.8)
- moved C18 1.84 mm to (134.9, 108.7)
- moved Y3 1.22 mm to (135.7, 105.7), turned to -90 degrees
- moved C25 1.20 mm to (132.9, 104.3), turned to 90 degrees
- moved C26 0.67 mm to (132.9, 107.0), turned to 90 degrees
Connections:
- IC4 pad 116: unconnected-(IC4-PD2-Pad116) -> LED_CAM
Routing:
- net LED_CAM: track 0.00 -> 7.40 mm
- net Net-(J9-Pin_2): track 0.00 -> 2.21 mm
- net +3V3: track 76.1 -> 78.2 mm
- net PH0-OSC_IN: track 7.20 -> 8.70 mm
- net DIN Board 1: track 43.4 -> 44.5 mm
- net GND: vias 88 -> 96
