File: PCB/front/front.kicad_pcb (KiCad board)
At the start: 2 copper layers, 43 x 26 mm, 22 parts, among them J1 Conn_01x06_Pin, J2 Conn_01x06_Pin, J3 Conn_01x08_Pin, U1 VL53L1CXV0FY1

Commit message: STM32 Mainboard requirements for Programing and Power
Changed lines of the file:
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@@
 		)
 		(property "Value" "VL53L1CXV0FY1"
-			(at -0.2 -2.6 -0)
+			(at -0.2 -2.6 0)
 			(layer "F.Fab")
 			(effects
@@
 	)
 	(segment
-		(start 89 129.125)
-		(end 89 128)
+		(start 89 128)
+		(end 88.5 127.5)
 		(width 0.25)
 		(layer "F.Cu")
@@
 	)
 	(segment
-		(start 89 128)
-		(end 88.5 127.5)
-		(width 0.25)
-		(layer "F.Cu")
-		(net 5)
-	)
-	(segment
 		(start 88.5875 121.8)
 		(end 88.5875 124.3)
@@
 	)
 	(segment
+		(start 89 129.125)
+		(end 89 128)
+		(width 0.25)
+		(layer "F.Cu")
+		(net 5)
+	)
+	(segment
 		(start 88.5 128.625)
 		(end 88.5 127.5)
@@
 	)
 	(segment
-		(start 91 126.25)
-		(end 91 127.773108)
+		(start 90.5 127.5)
+		(end 90.5 129.125)
 		(width 0.25)
 		(layer "F.Cu")
@@
 	)
 	(segment
-		(start 91 127.773108)
-		(end 90.5 128.273108)
+		(start 91 126.25)
+		(end 91 127)
 		(width 0.25)
 		(layer "F.Cu")
@@
 	)
 	(segment
-		(start 90.5 128.273108)
-		(end 90.5 129.125)
+		(start 91 127)
+		(end 90.5 127.5)
 		(width 0.25)
 		(layer "F.Cu")
@@
 	)
 	(segment
-		(start 91 129.125)
-		(end 91 128.410918)
+		(start 91 127.75)
+		(end 91.800003 126.949997)
 		(width 0.25)
 		(layer "F.Cu")
@@
 	)
 	(segment
-		(start 91.800003 127.610915)
-		(end 91.800003 126.25)
+		(start 91 129.125)
+		(end 91 127.75)
 		(width 0.25)
 		(layer "F.Cu")
@@
 	)
 	(segment
-		(start 91 128.410918)
-		(end 91.800003 127.610915)
+		(start 91.800003 126.949997)
+		(end 91.800003 126.25)
 		(width 0.25)
 		(layer "F.Cu")
@@
 	)
 	(segment
-		(start 90 128.107772)
-		(end 90 129.125)
+		(start 90.107772 127.142228)
+		(end 90 127.25)
 		(width 0.25)
 		(layer "F.Cu")
@@
 	)
 	(segment
-		(start 90.107772 128)
-		(end 90 128.107772)
+		(start 90 127.25)
+		(end 90 129.125)
 		(width 0.25)
 		(layer "F.Cu")
@@
 	(segment
 		(start 90.107772 126.25)
-		(end 90.107772 128)
+		(end 90.107772 127.142228)
 		(width 0.25)
 		(layer "F.Cu")
@@
 	)
 	(segment
-		(start 89.481772 129.106772)
-		(end 89.5 129.125)
+		(start 89.25 127)
+		(end 89.481772 127.231772)
 		(width 0.25)
 		(layer "F.Cu")
@@
 	(segment
 		(start 89.25 126.307769)
-		(end 89.25 127.61219)
+		(end 89.25 127)
 		(width 0.25)
 		(layer "F.Cu")
@@
 	)
 	(segment
-		(start 89.25 127.61219)
-		(end 89.481772 127.843962)
+		(start 89.481772 129.106772)
+		(end 89.5 129.125)
 		(width 0.25)
 		(layer "F.Cu")
@@
 	)
 	(segment
-		(start 89.481772 127.843962)
+		(start 89.481772 127.231772)
 		(end 89.481772 129.106772)
 		(width 0.25)

Commit message: random upload
Parts:
- C1, C2, C3, C4, C5, C6, C7, C8: footprint Capacitor_SMD:C_1206_3216Metric_Pad1.33x1.80mm_HandSolder -> Capacitor_SMD:C_0402_1005Metric_Pad0.74x0.62mm_HandSolder
- J1, J2: footprint Connector_FFC-FPC:Amphenol_F32Q-1A7x1-11006_1x06-1MP_P0.5mm_Horizontal -> Library:849526
- J3: footprint Connector_FFC-FPC:Amphenol_F32Q-1A7x1-11008_1x08-1MP_P0.5mm_Horizontal -> Library:17352658
- moved J3 0.32 mm to (90.3, 131.7)
- moved J1 0.25 mm to (75.8, 122.0)
- moved J2 0.25 mm to (61.0, 122.0)
Routing:
- net 3.3V: track 13.9 -> 3.50 mm
- net GND Board 2: track 30.6 -> 25.3 mm, vias 4 -> 5
- net DIN Board 1: track 15.6 -> 18.8 mm
- net 5V Board 1: track 7.10 -> 5.37 mm, vias 4 -> 3
- net DIN Board 2: track 15.7 -> 16.8 mm
- net XSHUT: track 10.8 -> 9.82 mm
- net Net-(D2-DOUT): track 7.58 -> 8.37 mm
- net SCL: track 3.95 -> 3.21 mm
- net GND Board 1: track 24.2 -> 23.6 mm
- net SDA: track 3.79 -> 3.25 mm
- net 5V Board 2: track 5.64 -> 5.28 mm, vias 4 -> 2
- net GND: track 4.17 -> 4.16 mm, vias 5 -> 4
Other:
- outline, holes or cut-outs redrawn

Commit message: random
Parts:
- moved C2 72.5 mm to (143.3, 105.3)
- moved C3 72.5 mm to (143.3, 97.1)
- moved C7 72.5 mm to (156.9, 93.6)
- moved C8 72.5 mm to (156.9, 96.1)
- moved D2 72.5 mm to (143.4, 93.1)
- moved D3 72.5 mm to (143.4, 101.2)
- moved D4 72.5 mm to (126.6, 84.6)
- moved D6 72.5 mm to (126.5, 101.0)
- moved J3 72.5 mm to (157.0, 103.5)
- moved TP1 72.5 mm to (135.0, 82.9)
- moved TP2 72.5 mm to (135.0, 104.8)
- moved TP3 72.5 mm to (148.0, 104.8)
- moved TP4 72.5 mm to (148.0, 91.8)
- moved U1 72.5 mm to (156.9, 96.4)
- moved C1 72.5 mm to (143.3, 88.9)
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